File: hw/scorzonera.sch (KiCad schematic (older format))
At the start: 7 parts, among them J1 NEIGHBOR1, J2 NEIGHBOR2, J7 BONUS_ROW

Commit message: Fix up schematic libs & symbols
Parts:
- J1, J2: symbol CONN_02X20 -> Connector_Generic:Conn_02x20_Odd_Even
- J7: symbol CONN_01X20 -> Connector_Generic:Conn_01x20
- MH1, MH2, MH3, MH4: symbol CONN_01X01 -> Connector_Generic:Conn_01x01
Changed lines of the file:
@@
-EESchema Schematic File Version 2
-LIBS:power
-LIBS:device
-LIBS:transistors
-LIBS:conn
-LIBS:linear
-LIBS:regul
-LIBS:74xx
-LIBS:cmos4000
-LIBS:adc-dac
-LIBS:memory
-LIBS:xilinx
-LIBS:microcontrollers
-LIBS:dsp
-LIBS:microchip
-LIBS:analog_switches
-LIBS:motorola
-LIBS:texas
-LIBS:intel
-LIBS:audio
-LIBS:interface
-LIBS:digital-audio
-LIBS:philips
-LIBS:display
-LIBS:cypress
-LIBS:siliconi
-LIBS:opto
-LIBS:atmel
-LIBS:contrib
-LIBS:valves
-LIBS:gsg-symbols
-LIBS:scorzonera-cache
-EELAYER 25 0
+EESchema Schematic File Version 4
+EELAYER 26 0
 EELAYER END
 $Descr USLedger 17000 11000
@@
 P2_8
 $Comp
-L CONN_02X20 J2
+L Connector_Generic:Conn_02x20_Odd_Even J2
 U 1 1 55EAB4B7
-P 15750 2900
-F 0 "J2" H 15750 3950 50  0000 C CNN
-F 1 "NEIGHBOR2" V 15750 2900 50  0000 C CNN
-F 2 "gsg-modules:HEADER-2x20" H 15750 1950 60  0001 C CNN
-F 3 "" H 15750 1950 60  0000 C CNN
-F 4 "Samtec" H 15750 2900 60  0001 C CNN "Manufacturer"
-F 5 "SSQ-120-23-G-D" H 15750 2900 60  0001 C CNN "Part Number"
-F 6 "CONN RCPT .100\" 40POS DUAL-ROW STACKING GOLD" H 15750 2900 60  0001 C CNN "Description"
-F 7 "Alternate: https://www.adafruit.com/products/2223" H 15750 2900 60  0001 C CNN "Note"
-	1    15750 2900
-	1    0    0    -1
-$EndComp
-$Comp
-L GND #PWR059
+P 15700 2850
+F 0 "J2" H 15700 3900 50  0000 C CNN
+F 1 "NEIGHBOR2" V 15700 2850 50  0000 C CNN
+F 2 "gsg-modules:HEADER-2x20" H 15700 1900 60  0001 C CNN
+F 3 "" H 15700 1900 60  0000 C CNN
+F 4 "Samtec" H 15700 2850 60  0001 C CNN "Manufacturer"
+F 5 "SSQ-120-23-G-D" H 15700 2850 60  0001 C CNN "Part Number"
+F 6 "CONN RCPT .100\" 40POS DUAL-ROW STACKING GOLD" H 15700 2850 60  0001 C CNN "Description"
+F 7 "Alternate: https://www.adafruit.com/products/2223" H 15700 2850 60  0001 C CNN "Note"
+	1    15700 2850
+	1    0    0    -1
+$EndComp
+$Comp
+L power:GND #PWR059
 U 1 1 55EACE84
 P 15300 1950
@@
 $EndComp
 $Comp
-L GND #PWR060
+L power:GND #PWR060
 U 1 1 55EAECD0
 P 15300 4300
@@
 $EndComp
 $Comp
-L VCC #PWR061
+L power:VCC #PWR061
 U 1 1 55EAF03E
 P 16200 4300
@@
 VBUS
 $Comp
-L CONN_02X20 J1
+L Connector_Generic:Conn_02x20_Odd_Even J1
 U 1 1 55FB1D52
-P 15750 5250
-F 0 "J1" H 15750 6300 50  0000 C CNN
-F 1 "NEIGHBOR1" V 15750 5250 50  0000 C CNN
-F 2 "gsg-modules:HEADER-2x20" H 15750 4300 60  0001 C CNN
-F 3 "" H 15750 4300 60  0000 C CNN
-F 4 "Samtec" H 15750 5250 60  0001 C CNN "Manufacturer"
-F 5 "SSQ-120-23-G-D" H 15750 5250 60  0001 C CNN "Part Number"
-F 6 "CONN RCPT .100\" 40POS DUAL-ROW STACKING GOLD" H 15750 5250 60  0001 C CNN "Description"
-F 7 "Alternate: https://www.adafruit.com/products/2223" H 15750 5250 60  0001 C CNN "Note"
-	1    15750 5250
+P 15700 5200
+F 0 "J1" H 15700 6250 50  0000 C CNN
+F 1 "NEIGHBOR1" V 15700 5200 50  0000 C CNN
+F 2 "gsg-modules:HEADER-2x20" H 15700 4250 60  0001 C CNN
+F 3 "" H 15700 4250 60  0000 C CNN
+F 4 "Samtec" H 15700 5200 60  0001 C CNN "Manufacturer"
+F 5 "SSQ-120-23-G-D" H 15700 5200 60  0001 C CNN "Part Number"
+F 6 "CONN RCPT .100\" 40POS DUAL-ROW STACKING GOLD" H 15700 5200 60  0001 C CNN "Description"
+F 7 "Alternate: https://www.adafruit.com/products/2223" H 15700 5200 60  0001 C CNN "Note"
+	1    15700 5200
 	1    0    0    -1
 $EndComp
@@
 P2_13
 $Comp
-L GND #PWR075
+L power:GND #PWR075
 U 1 1 560E00A9
 P 14250 7550
@@
 $EndComp
 $Comp
-L VCC #PWR076
+L power:VCC #PWR076
 U 1 1 560E046D
 P 16150 7400
@@
 	16150 7400 16150 7200
 $Comp
-L CONN_01X20 J7
+L Connector_Generic:Conn_01x20 J7
 U 1 1 560E713A
-P 15200 7000
-F 0 "J7" H 15200 8050 50  0000 C CNN
-F 1 "BONUS_ROW" V 15300 7000 50  0000 C CNN
-F 2 "gsg-modules:HEADER-1x20" H 15200 7000 60  0001 C CNN
-F 3 "" H 15200 7000 60  0000 C CNN
-F 4 "Samtec" H 15200 7000 60  0001 C CNN "Manufacturer"
-F 5 "SSQ-120-23-G-S" H 15200 7000 60  0001 C CNN "Part Number"
-F 6 "CONN RCPT .100\" 20POS SINGLE-ROW STACKING GOLD" H 15200 7000 60  0001 C CNN "Description"
-F 7 "DNP" V 15400 7000 60  0000 C CNN "Note"
-	1    15200 7000
+P 15150 7000
+F 0 "J7" H 15150 8050 50  0000 C CNN
+F 1 "BONUS_ROW" V 15250 7000 50  0000 C CNN
+F 2 "gsg-modules:HEADER-1x20" H 15150 7000 60  0001 C CNN
+F 3 "" H 15150 7000 60  0000 C CNN
+F 4 "Samtec" H 15150 7000 60  0001 C CNN "Manufacturer"
+F 5 "SSQ-120-23-G-S" H 15150 7000 60  0001 C CNN "Part Number"
+F 6 "CONN RCPT .100\" 20POS SINGLE-ROW STACKING GOLD" H 15150 7000 60  0001 C CNN "Description"
+F 7 "DNP" V 15350 7000 60  0000 C CNN "Note"
+	1    15150 7000
 	0    -1   -1   0
 $EndComp
@@
 ADC0_5
 $Comp
-L CONN_01X01 MH3
+L Connector_Generic:Conn_01x01 MH3
 U 1 1 5600EED5
 P 13650 850
@@
 $EndComp
 $Comp
-L GND #PWR077
+L power:GND #PWR077
 U 1 1 5600F9D3
 P 13650 1150
@@
 	13650 1050 13650 1150
 $Comp
-L CONN_01X01 MH4
+L Connector_Generic:Conn_01x01 MH4
 U 1 1 560100F3
 P 14150 1000
@@
 $EndComp
 $Comp
-L GND #PWR078
+L power:GND #PWR078
 U 1 1 560100F9
 P 14150 1300
@@
 	14150 1200 14150 1300
 $Comp
-L CONN_01X01 MH1
+L Connector_Generic:Conn_01x01 MH1
 U 1 1 56010ADB
 P 12650 850
@@
 $EndComp
 $Comp
-L GND #PWR079
+L power:GND #PWR079
 U 1 1 56010AE1
 P 12650 1150
@@
 	12650 1050 12650 1150
 $Comp
-L CONN_01X01 MH2
+L Connector_Generic:Conn_01x01 MH2
 U 1 1 56010AE9
 P 13150 1000
@@
 $EndComp
 $Comp
-L GND #PWR080
+L power:GND #PWR080
 U 1 1 56010AEF
 P 13150 1300
@@
 	16050 7550 16050 7200
 $Comp
-L GND #PWR081
+L power:GND #PWR081
 U 1 1 56035FE9
 P 16050 7550
@@
 	15150 7550 15150 7200
 $Comp
-L GND #PWR082
+L power:GND #PWR082
 U 1 1 56036BE7
 P 15150 7550
