File: hw/scorzonera.sch (KiCad schematic (older format))
At the start: 7 parts, among them J1 NEIGHBOR1, J2 NEIGHBOR2, J7 BONUS_ROW

Commit message: Add AM7969 symbol
Parts:
- added U?: AM7969, symbol Interface:AM7969
Changed lines of the file:
@@
+	1    0    0    -1
+$EndComp
+$Comp
+L Interface:AM7969 U?
+U 1 1 5CCFE902
+P 4250 3750
+F 0 "U?" H 4250 5028 50  0000 C CNN
+F 1 "AM7969" H 4250 4937 50  0000 C CNN
+F 2 "" H 4250 4150 50  0001 C CNN
+F 3 "" H 4250 4150 50  0001 C CNN
+	1    4250 3750
 	1    0    0    -1
 $EndComp

Commit message: Some wiring
Parts:
- added J?: Conn_01x02, symbol Connector_Generic:Conn_01x02
- U1: renamed from U?; footprint (none) -> Package_LCC:PLCC-28
Connections:
- net labels added: +5V, SGPIO0, SGPIO1, SGPIO10, SGPIO11, SGPIO12, SGPIO13, SGPIO14, SGPIO15, SGPIO2, SGPIO3, SGPIO4, SGPIO5, SGPIO6, SGPIO7, SGPIO8, SGPIO9
- net labels removed: P0_0, P0_1, P1_15, P1_16, P6_6, P6_7, P6_8, P7_0
- wire segments 103 -> 119
- no-connect marks 0 -> 2
Other:
- note added: "TODO:\nAdd level translator\nPick pins for SGPIO[8..15]\nPick XTAL & add"

Commit message: Map out remaining SGPIO, add SERIN dividers, etc.
Parts:
- added R1, R3: 120R, Resistor_SMD:R_0603_1608Metric, symbol Device:R
- added R2, R4: 330R, Resistor_SMD:R_0603_1608Metric, symbol Device:R
- J3: renamed from J?; footprint (none) -> Connector_PinHeader_2.54mm:PinHeader_1x02_P2.54mm_Vertical
Connections:
- net labels added: SERIN+, SERIN-
- net labels removed: P4_10, P4_2, P4_3, P4_4, P4_5, P4_6, P4_8, P4_9
- wire segments 119 -> 123
Other:
- note added: "TODO:\nAdd level translator\nPick XTAL & add\nAdd RS232 stuff"
- note removed: "TODO:\nAdd level translator\nPick pins for SGPIO[8..15]\nPick XTAL & add"
Changed lines of the file:
@@
 SGPIO0
 Text Label 9350 5350 0    40   ~ 0
-P4_9
+SGPIO14
 Text Label 10250 5450 2    40   ~ 0
 SGPIO1
 Text Label 9350 5450 0    40   ~ 0
-P4_10
+SGPIO15
 Text Label 10250 5550 2    40   ~ 0
 P5_0
@@
 ADC0_0
 Text Label 9350 3300 0    40   ~ 0
-P4_3
+SGPIO9
 Text Label 10250 3200 2    40   ~ 0
-P4_2
+SGPIO8
 Text Label 9350 3200 0    40   ~ 0
-P4_4
+SGPIO10
 Text Label 10250 3100 2    40   ~ 0
-P4_5
+SGPIO11
 Text Label 10250 3300 2    40   ~ 0
-P4_6
+SGPIO12
 Text Label 9350 3400 0    40   ~ 0
 P4_7
 Text Label 9350 3000 0    40   ~ 0
-P4_8
+SGPIO13
 Text Label 9250 3700 0    40   ~ 0
 WAKEUP0
@@
 SGPIO15
 $Comp
-L Connector_Generic:Conn_01x02 J?
+L Connector_Generic:Conn_01x02 J3
 U 1 1 5CD3D07A
-P 4400 4850
-F 0 "J?" H 4320 4525 50  0000 C CNN
-F 1 "Conn_01x02" H 4320 4616 50  0000 C CNN
-F 2 "" H 4400 4850 50  0001 C CNN
-F 3 "~" H 4400 4850 50  0001 C CNN
-	1    4400 4850
+P 2600 4850
+F 0 "J3" H 2520 4525 50  0000 C CNN
+F 1 "Conn_01x02" H 2520 4616 50  0000 C CNN
+F 2 "Connector_PinHeader_2.54mm:PinHeader_1x02_P2.54mm_Vertical" H 2600 4850 50  0001 C CNN
+F 3 "~" H 2600 4850 50  0001 C CNN
+	1    2600 4850
 	-1   0    0    1
 $EndComp
-Wire Wire Line
-	4600 4750 4850 4750
-Wire Wire Line
-	4850 4850 4600 4850
 Text Notes 11250 4200 0    200  ~ 0
-TODO:\nAdd level translator\nPick pins for SGPIO[8..15]\nPick XTAL & add
+TODO:\nAdd level translator\nPick XTAL & add\nAdd RS232 stuff
 Wire Wire Line
 	6050 5950 6050 6850
@@
 Wire Wire Line
 	4650 5350 4850 5350
+Text Label 4850 4750 2    50   ~ 0
+SERIN+
+Text Label 4850 4850 2    50   ~ 0
+SERIN-
+$Comp
+L Device:R R1
+U 1 1 5CD51D8E
+P 3200 4550
+F 0 "R1" H 3270 4596 50  0000 L CNN
+F 1 "120R" H 3270 4505 50  0000 L CNN
+F 2 "Resistor_SMD:R_0603_1608Metric" V 3130 4550 50  0001 C CNN
+F 3 "~" H 3200 4550 50  0001 C CNN
+	1    3200 4550
+	1    0    0    -1
+$EndComp
+$Comp
+L Device:R R2
+U 1 1 5CD51DD4
+P 3200 5050
+F 0 "R2" H 3270 5096 50  0000 L CNN
+F 1 "330R" H 3270 5005 50  0000 L CNN
+F 2 "Resistor_SMD:R_0603_1608Metric" V 3130 5050 50  0001 C CNN
+F 3 "~" H 3200 5050 50  0001 C CNN
+	1    3200 5050
+	1    0    0    -1
+$EndComp
+$Comp
+L power:+5V #PWR0103
+U 1 1 5CD51E12
+P 3200 4400
+F 0 "#PWR0103" H 3200 4250 50  0001 C CNN
+F 1 "+5V" H 3215 4573 50  0000 C CNN
+F 2 "" H 3200 4400 50  0001 C CNN
+F 3 "" H 3200 4400 50  0001 C CNN
+	1    3200 4400
+	1    0    0    -1
+$EndComp
+$Comp
+L power:GND #PWR0104
+U 1 1 5CD51E33
+P 3200 5200
+F 0 "#PWR0104" H 3200 4950 50  0001 C CNN
+F 1 "GND" H 3205 5027 50  0000 C CNN
+F 2 "" H 3200 5200 50  0001 C CNN
+F 3 "" H 3200 5200 50  0001 C CNN
+	1    3200 5200
+	1    0    0    -1
+$EndComp
+$Comp
+L Device:R R3
+U 1 1 5CD51F2F
+P 3600 4550
+F 0 "R3" H 3670 4596 50  0000 L CNN
+F 1 "120R" H 3670 4505 50  0000 L CNN
+F 2 "Resistor_SMD:R_0603_1608Metric" V 3530 4550 50  0001 C CNN
+F 3 "~" H 3600 4550 50  0001 C CNN
+	1    3600 4550
+	1    0    0    -1
+$EndComp
+$Comp
+L Device:R R4
+U 1 1 5CD51F35
+P 3600 5050
+F 0 "R4" H 3670 5096 50  0000 L CNN
+F 1 "330R" H 3670 5005 50  0000 L CNN
+F 2 "Resistor_SMD:R_0603_1608Metric" V 3530 5050 50  0001 C CNN
+F 3 "~" H 3600 5050 50  0001 C CNN
+	1    3600 5050
+	1    0    0    -1
+$EndComp
+$Comp
+L power:+5V #PWR0105
+U 1 1 5CD51F3B
+P 3600 4400
+F 0 "#PWR0105" H 3600 4250 50  0001 C CNN
+F 1 "+5V" H 3615 4573 50  0000 C CNN
+F 2 "" H 3600 4400 50  0001 C CNN
+F 3 "" H 3600 4400 50  0001 C CNN
+	1    3600 4400
+	1    0    0    -1
+$EndComp
+$Comp
+L power:GND #PWR0106
+U 1 1 5CD51F41
+P 3600 5200
+F 0 "#PWR0106" H 3600 4950 50  0001 C CNN
+F 1 "GND" H 3605 5027 50  0000 C CNN
+F 2 "" H 3600 5200 50  0001 C CNN
+F 3 "" H 3600 5200 50  0001 C CNN
+	1    3600 5200
+	1    0    0    -1
+$EndComp
+Wire Wire Line
+	2800 4750 3200 4750
+Wire Wire Line
+	3200 4750 3200 4700
+Wire Wire Line
+	2800 4850 3600 4850
+Wire Wire Line
+	3200 4750 3200 4900
+Connection ~ 3200 4750
+Wire Wire Line
+	3600 4850 3600 4700
+Connection ~ 3600 4850
+Wire Wire Line
+	3600 4900 3600 4850
+Text Label 2800 4750 0    50   ~ 0
+SERIN+
+Text Label 2800 4850 0    50   ~ 0
+SERIN-
 $EndSCHEMATC

Commit message: Level translator and some routing
Parts:
- added U2: 74ALVC164245, Package_SO:TSSOP-48_6.1x12.5mm_P0.5mm, symbol Interface:74ALVC164245
Connections:
- net labels added: CLK, CO0, CO1, CO2, CO3, CSTRB, DO0, DO1, DO2, DO3, DO4, DO5, DO6, DO7, DSTRB, VLTN
- wire segments 123 -> 150
Other:
- note added: "TODO:\nPick XTAL & add\nAdd RS232 stuff"
- note removed: "TODO:\nAdd level translator\nPick XTAL & add\nAdd RS232 stuff"
Changed lines of the file:
@@
 	0    1    1    0
 $EndComp
-Text Label 10250 2900 2    40   ~ 0
-VBUS
 $Comp
 L Connector_Generic:Conn_02x20_Odd_Even J1
@@
 	9350 5350 9550 5350
 Wire Wire Line
-	9350 2900 9550 2900
+	9350 2900 9450 2900
 Wire Wire Line
 	9350 5450 9550 5450
@@
 	1    0    0    -1
 $EndComp
-Text Label 6050 4250 0    50   ~ 0
+Text Label 7350 4250 0    50   ~ 0
 SGPIO0
-Text Label 6050 4350 0    50   ~ 0
+Text Label 7350 4350 0    50   ~ 0
 SGPIO1
-Text Label 6050 4450 0    50   ~ 0
+Text Label 7350 4450 0    50   ~ 0
 SGPIO2
-Text Label 6050 4550 0    50   ~ 0
+Text Label 7350 4550 0    50   ~ 0
 SGPIO3
-Text Label 6050 4650 0    50   ~ 0
+Text Label 7350 4650 0    50   ~ 0
 SGPIO4
-Text Label 6050 4750 0    50   ~ 0
+Text Label 7350 4750 0    50   ~ 0
 SGPIO5
-Text Label 6050 4850 0    50   ~ 0
+Text Label 7350 4850 0    50   ~ 0
 SGPIO6
-Text Label 6050 4950 0    50   ~ 0
+Text Label 7350 4950 0    50   ~ 0
 SGPIO7
 NoConn ~ 4850 5550
@@
 	5500 3850 5550 3850
 NoConn ~ 6050 5850
-Text Label 6050 5650 0    50   ~ 0
+Text Label 7350 5550 0    50   ~ 0
 SGPIO8
-Text Label 6050 5750 0    50   ~ 0
+Text Label 7350 5650 0    50   ~ 0
 SGPIO9
-Text Label 6050 5950 0    50   ~ 0
+Text Label 7350 5750 0    50   ~ 0
 SGPIO10
-Text Label 6050 5550 0    50   ~ 0
+Text Label 7350 5450 0    50   ~ 0
 SGPIO11
-Text Label 6050 5050 0    50   ~ 0
+Text Label 7350 5350 0    50   ~ 0
 SGPIO12
-Text Label 6050 5150 0    50   ~ 0
+Text Label 7350 5250 0    50   ~ 0
 SGPIO13
-Text Label 6050 5250 0    50   ~ 0
+Text Label 7350 5150 0    50   ~ 0
 SGPIO14
-Text Label 6050 5350 0    50   ~ 0
+Text Label 7350 5050 0    50   ~ 0
 SGPIO15
 $Comp
@@
 $EndComp
 Text Notes 11250 4200 0    200  ~ 0
-TODO:\nAdd level translator\nPick XTAL & add\nAdd RS232 stuff
-Wire Wire Line
-	6050 5950 6050 6850
-Wire Wire Line
-	6050 6850 4650 6850
-Wire Wire Line
-	4650 6850 4650 5350
-Wire Wire Line
-	4650 5350 4850 5350
+TODO:\nPick XTAL & add\nAdd RS232 stuff
 Text Label 4850 4750 2    50   ~ 0
 SERIN+
@@
 Text Label 2800 4850 0    50   ~ 0
 SERIN-
+$Comp
+L Interface:74ALVC164245 U2
+U 1 1 5CD8BD41
+P 6950 4950
+F 0 "U2" H 6950 6215 50  0000 C CNN
+F 1 "74ALVC164245" H 6950 6124 50  0000 C CNN
+F 2 "Package_SO:TSSOP-48_6.1x12.5mm_P0.5mm" H 6950 4950 50  0001 C CNN
+F 3 "" H 6950 4950 50  0001 C CNN
+	1    6950 4950
+	1    0    0    -1
+$EndComp
+Wire Wire Line
+	6050 4250 6550 4250
+Wire Wire Line
+	6550 4350 6050 4350
+Wire Wire Line
+	6050 4450 6550 4450
+Wire Wire Line
+	6550 4550 6050 4550
+Wire Wire Line
+	6050 4650 6550 4650
+Wire Wire Line
+	6550 4750 6050 4750
+Wire Wire Line
+	6050 4850 6550 4850
+Wire Wire Line
+	6550 4950 6050 4950
+Wire Wire Line
+	6050 5050 6550 5050
+Wire Wire Line
+	6550 5150 6050 5150
+Wire Wire Line
+	6050 5250 6550 5250
+Wire Wire Line
+	6550 5350 6050 5350
+Wire Wire Line
+	6050 5550 6100 5550
+Wire Wire Line
+	6100 5550 6100 5450
+Wire Wire Line
+	6100 5450 6550 5450
+Wire Wire Line
+	6050 5750 6200 5750
+Wire Wire Line
+	6050 5950 6250 5950
+Wire Wire Line
+	6250 5950 6250 5750
+Wire Wire Line
+	6250 5750 6550 5750
+Text Label 4850 5350 2    50   ~ 0
+CLK
+$Comp
+L power:GND #PWR0107
+U 1 1 5CE07E1C
+P 4600 5650
+F 0 "#PWR0107" H 4600 5400 50  0001 C CNN
+F 1 "GND" H 4605 5477 50  0000 C CNN
+F 2 "" H 4600 5650 50  0001 C CNN
+F 3 "" H 4600 5650 50  0001 C CNN
+	1    4600 5650
+	1    0    0    -1
+$EndComp
+Wire Wire Line
+	4850 5450 4600 5450
+Wire Wire Line
+	4600 5450 4600 5650
+Text Label 10050 2900 0    40   ~ 0
+VBUS
+$Comp
+L power:+5V #PWR0108
+U 1 1 5CE31150
+P 10250 2900
+F 0 "#PWR0108" H 10250 2750 50  0001 C CNN
+F 1 "+5V" V 10265 3028 50  0000 L CNN
+F 2 "" H 10250 2900 50  0001 C CNN
+F 3 "" H 10250 2900 50  0001 C CNN
+	1    10250 2900
+	0    1    1    0
+$EndComp
+Wire Wire Line
+	10250 2900 10050 2900
+$Comp
+L power:+5V #PWR0109
+U 1 1 5CE394DC
+P 6200 3850
+F 0 "#PWR0109" H 6200 3700 50  0001 C CNN
+F 1 "+5V" H 6215 4023 50  0000 C CNN
+F 2 "" H 6200 3850 50  0001 C CNN
+F 3 "" H 6200 3850 50  0001 C CNN
+	1    6200 3850
+	1    0    0    -1
+$EndComp
+Wire Wire Line
+	6200 3850 6200 3950
+Wire Wire Line
+	6200 3950 6550 3950
+$Comp
+L power:VCC #PWR0110
+U 1 1 5CE41ABC
+P 7400 3850
+F 0 "#PWR0110" H 7400 3700 50  0001 C CNN
+F 1 "VCC" H 7417 4023 50  0000 C CNN
+F 2 "" H 7400 3850 50  0001 C CNN
+F 3 "" H 7400 3850 50  0001 C CNN
+	1    7400 3850
+	1    0    0    -1
+$EndComp
+Wire Wire Line
+	7400 3850 7400 3950
+Wire Wire Line
+	7400 3950 7350 3950
+$Comp
+L power:GND #PWR0111
+U 1 1 5CE52F19
+P 6750 6150
+F 0 "#PWR0111" H 6750 5900 50  0001 C CNN
+F 1 "GND" H 6755 5977 50  0000 C CNN
+F 2 "" H 6750 6150 50  0001 C CNN
+F 3 "" H 6750 6150 50  0001 C CNN
+	1    6750 6150
+	1    0    0    -1
+$EndComp
+Wire Wire Line
+	6950 6050 6750 6150
+$Comp
+L power:PWR_FLAG #FLG0101
+U 1 1 5CE5BDA6
+P 9450 2900
+F 0 "#FLG0101" H 9450 2975 50  0001 C CNN
+F 1 "PWR_FLAG" H 9450 3074 50  0000 C CNN
+F 2 "" H 9450 2900 50  0001 C CNN
+F 3 "~" H 9450 2900 50  0001 C CNN
+	1    9450 2900
+	1    0    0    -1
+$EndComp
+Connection ~ 9450 2900
+Wire Wire Line
+	9450 2900 9550 2900
+Text Label 6050 4250 0    50   ~ 0
+DO0
+Text Label 6050 4350 0    50   ~ 0
+DO1
+Text Label 6050 4450 0    50   ~ 0
+DO2
+Text Label 6050 4550 0    50   ~ 0
+DO3
+Text Label 6050 4650 0    50   ~ 0
+DO4
+Text Label 6050 4750 0    50   ~ 0
+DO5
+Text Label 6050 4850 0    50   ~ 0
+DO6
+Text Label 6050 4950 0    50   ~ 0
+DO7
+Text Label 6050 5050 0    50   ~ 0
+CO3
+Text Label 6050 5150 0    50   ~ 0
+CO2
+Text Label 6050 5250 0    50   ~ 0
+CO1
+Text Label 6050 5350 0    50   ~ 0
+CO0
+Text Label 6100 5450 0    50   ~ 0
+VLTN
+Text Label 6250 5650 0    50   ~ 0
+DSTRB
+Text Label 6200 5550 0    50   ~ 0
+CSTRB
+Text Label 6250 5750 0    50   ~ 0
+CLK
+Wire Wire Line
+	6050 5650 6550 5650
+Wire Wire Line
+	6200 5750 6200 5550
+Wire Wire Line
+	6200 5550 6550 5550
 $EndSCHEMATC

Commit message: Routed! for now
Other:
- note added: "TODO:\nSprinkle caps everywhere\nPick XTAL & add\nAdd RS232 stuff"
- note removed: "TODO:\nPick XTAL & add\nAdd RS232 stuff"
Changed lines of the file:
@@
 EESchema Schematic File Version 4
+LIBS:scorzonera-cache
 EELAYER 26 0
 EELAYER END
@@
 $EndComp
 Text Notes 11250 4200 0    200  ~ 0
-TODO:\nPick XTAL & add\nAdd RS232 stuff
+TODO:\nSprinkle caps everywhere\nPick XTAL & add\nAdd RS232 stuff
 Text Label 4850 4750 2    50   ~ 0
 SERIN+

Commit message: RS232
Parts:
- added J4: Conn_01x02, Connector_PinHeader_2.54mm:PinHeader_1x02_P2.54mm_Vertical, symbol Connector_Generic:Conn_01x02
- added U3: MAX3232, Package_SO:TSSOP-16_4.4x5mm_P0.65mm, symbol Interface_UART:MAX3232
Connections:
- net labels added: U1_RXD, U1_TXD
- net labels removed: P3_4, P3_5
- wire segments 150 -> 156
Other:
- note added: "TODO:\nSprinkle caps everywhere\nPick XTAL & add"
- note removed: "TODO:\nSprinkle caps everywhere\nPick XTAL & add\nAdd RS232 stuff"
Changed lines of the file:
@@
 P3_3
 Text Label 10250 4200 2    40   ~ 0
-P3_4
+U1_TXD
 Text Label 9350 3900 0    40   ~ 0
 PF_4
 Text Label 9350 4700 0    40   ~ 0
-P3_5
+U1_RXD
 Text Label 10250 4700 2    40   ~ 0
 P3_6
@@
 $EndComp
 Text Notes 11250 4200 0    200  ~ 0
-TODO:\nSprinkle caps everywhere\nPick XTAL & add\nAdd RS232 stuff
+TODO:\nSprinkle caps everywhere\nPick XTAL & add
 Text Label 4850 4750 2    50   ~ 0
 SERIN+
@@
 Wire Wire Line
 	6200 5550 6550 5550
+$Comp
+L Interface_UART:MAX3232 U3
+U 1 1 5CD0B377
+P 6950 8100
+F 0 "U3" H 6500 9350 50  0000 C CNN
+F 1 "MAX3232" H 6600 9250 50  0000 C CNN
+F 2 "Package_SO:TSSOP-16_4.4x5mm_P0.65mm" H 7000 7050 50  0001 L CNN
+F 3 "https://datasheets.maximintegrated.com/en/ds/MAX3222-MAX3241.pdf" H 6950 8200 50  0001 C CNN
+	1    6950 8100
+	1    0    0    -1
+$EndComp
+$Comp
+L power:VCC #PWR01
+U 1 1 5CD0B752
+P 6950 6900
+F 0 "#PWR01" H 6950 6750 50  0001 C CNN
+F 1 "VCC" H 6950 7050 50  0000 C CNN
+F 2 "" H 6950 6900 60  0000 C CNN
+F 3 "" H 6950 6900 60  0000 C CNN
+	1    6950 6900
+	1    0    0    -1
+$EndComp
+$Comp
+L power:GND #PWR02
+U 1 1 5CD0BBF3
+P 6950 9300
+F 0 "#PWR02" H 6950 9050 50  0001 C CNN
+F 1 "GND" H 6950 9150 50  0000 C CNN
+F 2 "" H 6950 9300 60  0000 C CNN
+F 3 "" H 6950 9300 60  0000 C CNN
+	1    6950 9300
+	1    0    0    -1
+$EndComp
+Text Label 6150 8600 2    40   ~ 0
+U1_RXD
+Text Label 6150 8200 2    40   ~ 0
+U1_TXD
+$Comp
+L Connector_Generic:Conn_01x02 J4
+U 1 1 5CD0C913
+P 8900 8350
+F 0 "J4" H 8820 8025 50  0000 C CNN
+F 1 "Conn_01x02" H 8820 8116 50  0000 C CNN
+F 2 "Connector_PinHeader_2.54mm:PinHeader_1x02_P2.54mm_Vertical" H 8900 8350 50  0001 C CNN
+F 3 "~" H 8900 8350 50  0001 C CNN
+	1    8900 8350
+	1    0    0    -1
+$EndComp
+Wire Wire Line
+	7750 8200 8150 8200
+Wire Wire Line
+	7750 8600 8150 8600
+Wire Wire Line
+	8150 8200 8150 8350
+Wire Wire Line
+	8150 8350 8700 8350
+Wire Wire Line
+	8150 8600 8150 8450
+Wire Wire Line
+	8150 8450 8700 8450
 $EndSCHEMATC

Commit message: Add Wago connector, more routing
Parts:
- removed J3, J4: Conn_01x02, Connector_PinHeader_2.54mm:PinHeader_1x02_P2.54mm_Vertical, symbol Connector_Generic:Conn_01x02
- added C1, C2: C, Capacitor_SMD:C_0402_1005Metric, symbol Device:C
- added C3, C4, C5, C6, C7: 100n, Capacitor_SMD:C_0402_1005Metric, symbol Device:C
- added J3: Conn_01x05, wago:256-743-5, symbol Connector_Generic:Conn_01x05
- added Y1: Crystal_GND24, Crystal:Crystal_SMD_SeikoEpson_TSX3225-4Pin_3.2x2.5mm, symbol Device:Crystal_GND24
- R1, R2, R3, R4: footprint Resistor_SMD:R_0603_1608Metric -> Resistor_SMD:R_0402_1005Metric
- U1: symbol Interface:AM7969 -> scorzonera:AM7969
- U2: symbol Interface:74ALVC164245 -> scorzonera:74ALVC164245
Connections:
- net labels added: RS232_RX, RS232_TX, X1, X2
- wire segments 156 -> 170
Other:
- note added: "TODO:\nSprinkle caps everywhere"
- note removed: "TODO:\nSprinkle caps everywhere\nPick XTAL & add"

Commit message: Switch to 2 level shifters, caps, route, silk
Parts:
- removed U2: 74ALVC164245, Package_SO:TSSOP-48_6.1x12.5mm_P0.5mm, symbol scorzonera:74ALVC164245
- added C10, C12, C13, C8, C9: 100n, Capacitor_SMD:C_0402_1005Metric, symbol Device:C
- added C11: 1u, Capacitor_SMD:C_0603_1608Metric, symbol Device:C
- added U4, U5: TXS0108EPW, wago:Texas_R-PVQFN-N20_4.65x3.65x1mm, symbol Logic_LevelTranslator:TXS0108EPW
- C1, C2: value C -> 18p; MPN (none) -> CC0402JRNPO9BN180
- C3, C4, C5, C6, C7: MPN (none) -> GRM155R61A104KA01D
- R1, R3: MPN (none) -> RC0402FR-07120RL
- R2, R4: MPN (none) -> RC0402FR-07330RL
- U3: MPN (none) -> MAX3232CUE+T
Connections:
- net labels added: U0_RXD, U0_TXD, notSGPIO15
- net labels removed: P2_8, P9_5, P9_6
- wire segments 170 -> 143
