File: hw/scorzonera.sch (KiCad schematic (older format))
At the start: 30 parts, among them J1 NEIGHBOR1, J2 NEIGHBOR2, J3 Conn_01x05, J7 BONUS_ROW, U1 AM7969, U3 MAX3232, U4 TXS0108EPW, U5 TXS0108EPW, Y1 Crystal_GND24

Commit message: Connect OEs & add pulldowns, more silk, random cleanup
Parts:
- added R5, R6: 10K, Resistor_SMD:R_0402_1005Metric, symbol Device:R
Connections:
- wire segments 143 -> 144
- no-connect marks 2 -> 20
Other:
- note removed: "TODO:\nSprinkle caps everywhere"
Changed lines of the file:
@@
 	9350 5250 9550 5250
 Wire Wire Line
-	10050 5250 10250 5250
+	10050 5250 10150 5250
 Wire Wire Line
 	10250 5350 10050 5350
@@
 Text Label 9550 1200 0    50   ~ 0
 SGPIO15
-Text Notes 11250 4200 0    200  ~ 0
-TODO:\nSprinkle caps everywhere
 Text Label 4850 4750 2    50   ~ 0
 SERIN+
@@
 Text Label 7650 2400 2    40   ~ 0
 P6_5
+Text Label 5300 1900 2    50   ~ 0
+P5_2
+Text Label 7650 2000 2    50   ~ 0
+P6_4
+$Comp
+L Device:R R6
+U 1 1 5CD97869
+P 7000 2150
+F 0 "R6" H 7070 2196 50  0000 L CNN
+F 1 "10K" H 7070 2105 50  0000 L CNN
+F 2 "Resistor_SMD:R_0402_1005Metric" V 6930 2150 50  0001 C CNN
+F 3 "~" H 7000 2150 50  0001 C CNN
+F 4 "RC0402FR-0710KL" H 0   0   50  0001 C CNN "MPN"
+	1    7000 2150
+	1    0    0    -1
+$EndComp
+Text Label 7000 2000 2    50   ~ 0
+P6_4
+$Comp
+L power:GND #PWR0132
+U 1 1 5CD97935
+P 7000 2300
+F 0 "#PWR0132" H 7000 2050 50  0001 C CNN
+F 1 "GND" H 7005 2127 50  0000 C CNN
+F 2 "" H 7000 2300 50  0001 C CNN
+F 3 "" H 7000 2300 50  0001 C CNN
+	1    7000 2300
+	1    0    0    -1
+$EndComp
+$Comp
+L Device:R R5
+U 1 1 5CD97A6E
+P 6650 2500
+F 0 "R5" H 6720 2546 50  0000 L CNN
+F 1 "10K" H 6720 2455 50  0000 L CNN
+F 2 "Resistor_SMD:R_0402_1005Metric" V 6580 2500 50  0001 C CNN
+F 3 "~" H 6650 2500 50  0001 C CNN
+F 4 "RC0402FR-0710KL" H 0   0   50  0001 C CNN "MPN"
+	1    6650 2500
+	1    0    0    -1
+$EndComp
+$Comp
+L power:GND #PWR0133
+U 1 1 5CD97A75
+P 6650 2650
+F 0 "#PWR0133" H 6650 2400 50  0001 C CNN
+F 1 "GND" H 6655 2477 50  0000 C CNN
+F 2 "" H 6650 2650 50  0001 C CNN
+F 3 "" H 6650 2650 50  0001 C CNN
+	1    6650 2650
+	1    0    0    -1
+$EndComp
+Text Label 6650 2350 2    50   ~ 0
+P5_2
+NoConn ~ 14550 7200
+NoConn ~ 14650 7200
+NoConn ~ 14750 7200
+NoConn ~ 14850 7200
+NoConn ~ 14950 7200
+NoConn ~ 15050 7200
+NoConn ~ 15250 7200
+NoConn ~ 15350 7200
+NoConn ~ 15450 7200
+NoConn ~ 15550 7200
+NoConn ~ 15650 7200
+NoConn ~ 15750 7200
+NoConn ~ 15850 7200
+NoConn ~ 15950 7200
+$Comp
+L power:PWR_FLAG #FLG0102
+U 1 1 5CE0C245
+P 10150 5250
+F 0 "#FLG0102" H 10150 5325 50  0001 C CNN
+F 1 "PWR_FLAG" H 10150 5424 50  0000 C CNN
+F 2 "" H 10150 5250 50  0001 C CNN
+F 3 "~" H 10150 5250 50  0001 C CNN
+	1    10150 5250
+	1    0    0    -1
+$EndComp
+Connection ~ 10150 5250
+Wire Wire Line
+	10150 5250 10250 5250
+$Comp
+L power:PWR_FLAG #FLG0103
+U 1 1 5CE0C9F6
+P 10050 2900
+F 0 "#FLG0103" H 10050 2975 50  0001 C CNN
+F 1 "PWR_FLAG" H 10050 3074 50  0000 C CNN
+F 2 "" H 10050 2900 50  0001 C CNN
+F 3 "~" H 10050 2900 50  0001 C CNN
+	1    10050 2900
+	1    0    0    -1
+$EndComp
+Connection ~ 10050 2900
+$Comp
+L power:GND #PWR0134
+U 1 1 5CE0CFD2
+P 6150 8400
+F 0 "#PWR0134" H 6150 8150 50  0001 C CNN
+F 1 "GND" V 6155 8272 50  0000 R CNN
+F 2 "" H 6150 8400 50  0001 C CNN
+F 3 "" H 6150 8400 50  0001 C CNN
+	1    6150 8400
+	0    1    1    0
+$EndComp
+$Comp
+L power:GND #PWR0135
+U 1 1 5CE0D044
+P 7750 8800
+F 0 "#PWR0135" H 7750 8550 50  0001 C CNN
+F 1 "GND" V 7755 8672 50  0000 R CNN
+F 2 "" H 7750 8800 50  0001 C CNN
+F 3 "" H 7750 8800 50  0001 C CNN
+	1    7750 8800
+	0    -1   -1   0
+$EndComp
+NoConn ~ 7750 8400
+NoConn ~ 6150 8800
+NoConn ~ 7650 2100
+NoConn ~ 8450 2100
 $EndSCHEMATC
